Commit message: 3

File: urdf/fianl.urdf (robot description, URDF)
Before this commit: robot uav_arm_combo, 11 links, 10 joints
Links:
- link body: mass 2.8 -> 2.9
Joints:
- joint joint0: origin xyz=0.24042 -0.24042 0.0466 rpy=0 0 0 -> xyz=0.22981 -0.22981 0.0466 rpy=0 0 0
- joint joint1: origin xyz=-0.24042 0.24042 0.0466 rpy=0 0 0 -> xyz=-0.22981 0.22981 0.0466 rpy=0 0 0
- joint joint2: origin xyz=0.24042 0.24042 0.0466 rpy=0 0 0 -> xyz=0.22981 0.22981 0.0466 rpy=0 0 0
- joint joint3: origin xyz=-0.24042 -0.24042 0.0466 rpy=0 0 0 -> xyz=-0.22981 -0.22981 0.0466 rpy=0 0 0
